File: nrfled.sch (EAGLE design)
At the start: 65 parts, among them IC1 MEGA48/88/168-AU, IC2 MAX487CSA, IC3 LM3401, IC4 78L05SMD, IC5 LM3401, IC6 LM3401, IC7 LM3401, IC8 78L05SMD, Q1 20MHz, Q2 MOSFET-PCHANNEL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

Commit message: More connections and extension connector
Parts:
- removed C1, C2, C3: 100nF, SparkFun:CAP0402-CAP
- removed IC2: MAX487CSA, maxim:MAX481CSA
- added EXT: (no value), pinhead:PINHD-2X5
Connections:
- new net AIN0: EXT.5, IC1.ADC6
- new net AIN1: EXT.6, IC1.ADC7
- new net INT: EXT.3, IC1.PD3(INT1/OC2B/PCINT19)
- new net IO0: EXT.7, IC1.PD4(T0/XCK/PCINT20)
- new net IO1: EXT.8, IC1.PD6(AIN0/OC0A/PCINT22)
- new net IO2: EXT.9, IC1.PD7(AIN1/PCINT23)
- net +12V: now also EXT.4
- net +3V3: now also EXT.1
- net +5V: now also EXT.2; no longer C1.1, C2.1, C3.1, IC2P.VCC
- net GND: now also EXT.10; no longer C1.2, C2.2, C3.2, IC2P.GND
