File: nrfled.brd (EAGLE design)
At the start: 67.9 x 38.8 mm, 65 parts, among them IC1 MEGA48/88/168-AU, IC2 MAX487CSA, IC3 LM3401, IC4 78L05SMD, IC5 LM3401, IC6 LM3401, IC7 LM3401, IC8 78L05SMD, Q1 20MHz, Q2 MOSFET-PCHANNEL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

Commit message: More connections and extension connector
Parts:
- removed C1, C2, C3: 100nF, SparkFun:0402-CAP
- removed IC2: MAX487CSA, maxim:SO08
- added EXT: (no value), pinhead:2X05
Connections:
- new net AIN0: EXT.5, IC1.19
- new net AIN1: EXT.6, IC1.22
- new net INT: EXT.3, IC1.1
- new net IO0: EXT.7, IC1.2
- new net IO1: EXT.8, IC1.10
- new net IO2: EXT.9, IC1.11
- net +12V: now also EXT.4
- net +3V3: now also EXT.1
- net +5V: now also EXT.2; no longer C1.1, C2.1, C3.1, IC2.8
- net GND: now also EXT.10; no longer C1.2, C2.2, C3.2, IC2.5
Routing:
- net +5V: track 55.9 -> 48.6 mm
- net GND: track 33.0 -> 31.0 mm, vias 67 -> 42
Other:
- board text added: "4CH Radio LED-Controller"
- board text removed: "4CH LED-Controller"

Commit message: Placement of parts, begin routing
Parts:
- moved EXT 71.9 mm to (63.3, 8.40), turned to 270 degrees
- moved JP1 57.4 mm to (50.0, 7.80), turned to 90 degrees
- moved C17 44.4 mm to (43.3, 4.00)
- moved C16 44.0 mm to (39.8, 4.00)
- moved IC8 42.2 mm to (41.4, 7.60), turned to 90 degrees
- moved FTDI 27.5 mm to (2.80, 8.90), turned to 90 degrees
- moved C5 9.41 mm to (19.9, 7.39)
- moved Q1 9.41 mm to (21.3, 5.06)
- moved C13 9.41 mm to (11.4, 3.80)
- moved IC4 9.41 mm to (13.1, 7.30)
- moved C12 9.41 mm to (15.0, 4.00)
- moved C4 9.41 mm to (18.7, 5.01)
- moved IC1 9.41 mm to (28.2, 8.77)
- moved R1 9.41 mm to (39.2, 13.3)
Routing:
- net !RST: track 24.0 -> 52.4 mm, vias 1 -> 2
- net TXD: track 2.98 -> 27.5 mm
- net RXD: track 9.91 -> 28.2 mm
- net !RE: track 13.4 -> 0.09 mm, vias 2 -> 0
- net PW: track 27.6 -> 39.9 mm
- net +12V: track 169.7 -> 179.1 mm
- net PR: track 44.9 -> 36.6 mm
- net PG: track 32.4 -> 24.4 mm
- net +5V: track 48.6 -> 41.6 mm
- net N$27: track 2.91 -> 7.01 mm
- net PB: track 17.4 -> 21.1 mm
